File: Project_02/EAGLE/ACL_Rehab_Tracker.sch (EAGLE design)
At the start: 18 parts, among them U1 POCKETBEAGLE, U2 MPU-6050-A

Commit message: Final Project_02
Connections:
- new net N$3: U1.VOUT@2
- new net N$4: U1.VOUT@1
- net GND: no longer U1.GND@3, U1.GND@4, U1.GND@5
Changed lines of the file:
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@@
 <setting verticaltext="up"/>
 </settings>
-<grid distance="0.1" unitdist="inch" unit="inch" style="lines" multiple="1" display="yes" altdistance="0.01" altunitdist="inch" altunit="inch"/>
+<grid distance="0.1" unitdist="inch" unit="inch" style="lines" multiple="1" display="no" altdistance="0.01" altunitdist="inch" altunit="inch"/>
 <layers>
 <layer number="1" name="Top" color="4" fill="1" visible="no" active="no"/>
@@
 <part name="SUPPLY4" library="Project_02_EDES_301" deviceset="VDD_3P3V" device=""/>
 <part name="GND3" library="Project_02_EDES_301" deviceset="GND" device=""/>
-<part name="GND4" library="Project_02_EDES_301" deviceset="GND" device=""/>
 <part name="GND5" library="Project_02_EDES_301" deviceset="GND" device=""/>
 <part name="FUD1" library="Project_02_EDES_301" deviceset="FIDUCIAL" device=""/>
@@
 <attribute name="VALUE" x="205.74" y="119.38" size="1.778" layer="96" rot="R180"/>
 </instance>
-<instance part="GND4" gate="1" x="35.56" y="142.24" smashed="yes">
-<attribute name="VALUE" x="33.02" y="139.7" size="1.778" layer="96"/>
-</instance>
 <instance part="GND5" gate="1" x="185.42" y="180.34" smashed="yes">
 <attribute name="VALUE" x="182.88" y="177.8" size="1.778" layer="96"/>
@@
 <wire x1="111.76" y1="198.12" x2="124.46" y2="198.12" width="0.1524" layer="91"/>
 <wire x1="124.46" y1="198.12" x2="124.46" y2="213.36" width="0.1524" layer="91"/>
+<label x="127" y="200.66" size="1.778" layer="95"/>
 </segment>
 <segment>
@@
 <segment>
 <pinref part="GND2" gate="1" pin="GND"/>
-<pinref part="U1" gate="G$1" pin="GND@4"/>
-<wire x1="127" y1="144.78" x2="111.76" y2="144.78" width="0.1524" layer="91"/>
 <pinref part="U1" gate="G$1" pin="GND@2"/>
 <wire x1="111.76" y1="147.32" x2="127" y2="147.32" width="0.1524" layer="91"/>
 <wire x1="127" y1="147.32" x2="127" y2="144.78" width="0.1524" layer="91"/>
-<junction x="127" y="144.78"/>
-</segment>
-<segment>
-<pinref part="U1" gate="G$1" pin="GND@5"/>
-<pinref part="GND4" gate="1" pin="GND"/>
-<wire x1="50.8" y1="144.78" x2="35.56" y2="144.78" width="0.1524" layer="91"/>
-<pinref part="U1" gate="G$1" pin="GND@3"/>
-<wire x1="50.8" y1="147.32" x2="35.56" y2="147.32" width="0.1524" layer="91"/>
-<wire x1="35.56" y1="147.32" x2="35.56" y2="144.78" width="0.1524" layer="91"/>
-<junction x="35.56" y="144.78"/>
 </segment>
 <segment>
@@
 </segment>
 </net>
+<net name="N$3" class="0">
+<segment>
+<pinref part="U1" gate="G$1" pin="VOUT@2"/>
+<wire x1="111.76" y1="200.66" x2="116.84" y2="200.66" width="0.1524" layer="91"/>
+<label x="116.84" y="200.66" size="1.778" layer="95"/>
+</segment>
+</net>
+<net name="N$4" class="0">
+<segment>
+<pinref part="U1" gate="G$1" pin="VOUT@1"/>
+<wire x1="50.8" y1="200.66" x2="43.18" y2="200.66" width="0.1524" layer="91"/>
+<label x="43.18" y="200.66" size="1.778" layer="95"/>
+</segment>
+</net>
